File: kicad/PCB/PCB.kicad_sch (KiCad schematic)
At the start: 53 parts, among them J1 JST_2mm, J2 JST_2mm, J3 3.5mm, J5 3.5mm, J6 3.5mm, J7 3.5mm, J9 Selector_TC4420, Q1 IRL520N, SW1 SW_DIP_x03, U1 XIAO-RP2350-DIP, U2 AP2112K-3.3, U3 TB6612FNG, U4 TC4420

Commit message: Limpieza de archivos innecesarios de PCB y creacion de guia de enrutado
Parts:
- U1: footprint Seeed_Studio_XIAO_Series:XIAO-RP2350-DIP -> Jaguar_Custom:XIAO-RP2350-DIP
Connections:
- net NET_MOTOR_EN: now also U1.11 (D10); no longer U1.10 (D9)
- net NET_VENT: now also U1.10 (D9); no longer U1.11 (D10)
Changed lines of the file:
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@@
 		)
 	)
-	(label "NET_MOTOR_EN"
+	(label "NET_VENT"
 		(at 187.96 143.51 0)
 		(effects
@@
 		)
 	)
-	(label "NET_VENT"
+	(label "NET_MOTOR_EN"
 		(at 193.04 139.7 0)
 		(effects
@@
 			)
 		)
-		(property "Footprint" "Seeed_Studio_XIAO_Series:XIAO-RP2350-DIP"
+		(property "Footprint" "Jaguar_Custom:XIAO-RP2350-DIP"
 			(at 180.848 124.46 0)
 			(hide yes)

Commit message: Fix J5/J6 topology, add connector labels, verify ERC, fill title block
Parts:
- J5: renamed from J6; value 3.5mm -> Ventilador
- J6: renamed from J5; value 3.5mm -> 48V IN
- renumbered R_LED to R_LED1
Other:
- note added: "Default: 1-2 (Bypass MCU)"
- title: PCB -> Evaluación Técnica - Sistemas Embebidos
Changed lines of the file:
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@@
 	(paper "USLetter" portrait)
 	(title_block
-		(title "PCB")
-		(date "2026-07-01")
+		(title "Evaluación Técnica - Sistemas Embebidos")
+		(date "2026-06-30")
+		(rev "1.1.1")
 		(company "Jaguar MX")
+		(comment 1 "Ing. Jair Molina Arce")
+		(comment 2 "Ingeniero de Sistemas Embebidos Jr.")
+	)
+	(text "Default: 1-2 (Bypass MCU)"
+		(exclude_from_sim no)
+		(at 27.686 74.168 0)
+		(effects
+			(font
+				(size 1.27 1.27)
+			)
+			(justify left bottom)
+		)
 	)
 	(junction
@@
 	(wire
 		(pts
-			(xy 185.42 139.7) (xy 193.04 139.7)
+			(xy 185.42 139.7) (xy 189.23 139.7)
 		)
 		(stroke
@@
 	)
 	(label "NET_MOTOR_EN"
-		(at 193.04 139.7 0)
+		(at 189.23 139.7 0)
 		(effects
 			(font
@@
 		(dnp no)
 		(fields_autoplaced yes)
-		(property "Reference" "J5"
+		(property "Reference" "J6"
 			(at 22.86 60.96 0)
 			(show_name no)
@@
 			)
 		)
-		(property "Value" "3.5mm"
+		(property "Value" "48V IN"
 			(at 22.86 63.5 0)
 			(show_name no)
@@
 			(project "PCB"
 				(path "/656cb11c-c675-4e3a-bafd-60f129c2bd91"
-					(reference "J5")
+					(reference "J6")
 					(unit 1)
 				)
@@
 		(in_pos_files yes)
 		(dnp no)
-		(property "Reference" "R_LED"
+		(property "Reference" "R_LED1"
 			(at 62.484 125.984 0)
 			(show_name no)
@@
 			(project "PCB"
 				(path "/656cb11c-c675-4e3a-bafd-60f129c2bd91"
-					(reference "R_LED")
+					(reference "R_LED1")
 					(unit 1)
 				)
@@
 		(dnp no)
 		(property "Reference" "C10"
-			(at 147.32 87.63 0)
+			(at 145.288 89.408 0)
 			(show_name no)
 			(do_not_autoplace no)
@@
 		)
 		(property "Value" "100uF/63V"
-			(at 153.67 91.44 0)
+			(at 145.796 92.456 0)
 			(show_name no)
 			(do_not_autoplace no)
@@
 		(in_pos_files yes)
 		(dnp no)
-		(property "Reference" "J6"
+		(property "Reference" "J5"
 			(at 22.86 88.55 0)
 			(show_name no)
@@
 			)
 		)
-		(property "Value" "3.5mm"
+		(property "Value" "Ventilador"
 			(at 22.86 76.55 0)
 			(show_name no)
@@
 			(project "PCB"
 				(path "/656cb11c-c675-4e3a-bafd-60f129c2bd91"
-					(reference "J6")
+					(reference "J5")
 					(unit 1)
 				)
